Commit message: Progress on build a Gazebo model of BEN.

File: urdf/ben.urdf (robot description, URDF)
Before this commit: robot ben, 1 links, 0 joints
Links:
- added link imu_link, mass 617.732; collision mesh filename=package://ben_description/models/meshes/BEN_convex_hull.dae; visual mesh filename=package://ben_description/models/meshes/BEN_shell.dae
- link base_link: mass 2000 -> None; geometry 
Joints:
- added joint base_to_imu_joint: type fixed, parent base_link, child imu_link, origin xyz=0 0 0.65 rpy=0 0 0

Commit message: Rename package to ben_gazebo

File: urdf/ben.urdf (robot description, URDF)
Before this commit: robot ben, 2 links, 1 joints
Links:
- link imu_link: geometry collision mesh filename=package://ben_gazebo/models/meshes/BEN_convex_hull.dae; visual mesh filename=package://ben_gazebo/models/meshes/BEN_shell.dae

File: urdf/ben.xacro (robot description, xacro)
@@ -12,18 +12,18 @@
   <xacro:property name="namespace" value="$(arg namespace)" scope="global" />
   <!-- Include macros for dynamics plugins -->
-  <xacro:include filename="$(find ben_description)/urdf/ben_dynamics_plugin.xacro" />
+  <xacro:include filename="$(find ben_gazebo)/urdf/ben_dynamics_plugin.xacro" />
   <!-- Attach hydrodynamics plugin -->
   <xacro:usv_dynamics_gazebo name="ben_dynamics_plugin" />
-  <xacro:include filename="$(find ben_description)/urdf/sensors/ben_gps.xacro" />
+  <xacro:include filename="$(find ben_gazebo)/urdf/sensors/ben_gps.xacro" />
   <xacro:ben_gps name="gps_ben" x="-0.85" />
-  <xacro:include filename="$(find ben_description)/urdf/sensors/ben_imu.xacro" />
+  <xacro:include filename="$(find ben_gazebo)/urdf/sensors/ben_imu.xacro" />
   <xacro:ben_imu name="imu_ben" y="-0.2" />
-  <xacro:include filename="$(find ben_description)/urdf/sensors/lidar.xacro" />
+  <xacro:include filename="$(find ben_gazebo)/urdf/sensors/lidar.xacro" />
   <xacro:lidar name="lidar_ben" y="-0.3" type="16_beam"/>
-  <xacro:include filename="$(find ben_description)/urdf/sensors/ben_camera.xacro" />
+  <xacro:include filename="$(find ben_gazebo)/urdf/sensors/ben_camera.xacro" />
   <xacro:ben_camera name="front_camera" y="0.3" x="0.75" P="${radians(15)}" />
   <!-- Robot mesh -->
-  <xacro:include filename="$(find ben_description)/urdf/ben.urdf" />
+  <xacro:include filename="$(find ben_gazebo)/urdf/ben.urdf" />
   <!-- === Thruster === -->
-  <xacro:include filename="$(find ben_description)/urdf/ben_thruster.xacro" />
+  <xacro:include filename="$(find ben_gazebo)/urdf/ben_thruster.xacro" />
 </robot>

File: urdf/sensors/lidar.xacro (robot description, xacro)
@@ -1,5 +1,5 @@
 <?xml version="1.0" encoding="UTF-8"?>
 <robot xmlns:xacro="http://ros.org/wiki/xacro">
-  <xacro:include filename="$(find ben_description)/urdf/sensors/ben_3d_lidar.xacro"/>
+  <xacro:include filename="$(find ben_gazebo)/urdf/sensors/ben_3d_lidar.xacro"/>
   <xacro:macro name="lidar"
                params = "type:='16_beam'
