Commit message: Add thruster (the one from the WAM-V) to BEN.

File: urdf/ben.xacro (robot description, xacro)
@@ -7,3 +7,11 @@
   <!-- Robot mesh -->
   <xacro:include filename="$(find ben_description)/urdf/ben.urdf" />
+  <!-- Note: this is only used for some sensors that do not correctly use the
+  robotNamespace parameter -->
+  <xacro:arg name="namespace" default="ben"/>
+  <xacro:property name="namespace" value="$(arg namespace)" scope="global" />
+  <!-- === Thruster === -->
+  <xacro:arg name="thruster_namespace" default="thrusters/"/>
+  <xacro:property name="thruster_namespace" value="$(arg thruster_namespace)" scope="global" />
+  <xacro:include filename="$(find ben_description)/urdf/ben_thruster.xacro" />
 </robot>

Commit message: Add sensors, which are copied from wam-v, so not yet positioned for BEN.

File: urdf/ben.xacro (robot description, xacro)
@@ -1,17 +1,29 @@
 <?xml version="1.0"?>
 <robot xmlns:xacro="http://ros.org/wiki/xacro" name="ben">
+  <!-- Note: this is only used for some sensors that do not correctly use the
+  robotNamespace parameter -->
+  <xacro:arg name="namespace" default="ben"/>
+  <xacro:arg name="thruster_namespace" default="thrusters/"/>
+  <xacro:arg name="camera_namespace" default="cameras/"/>
+  <xacro:arg name="sensor_namespace" default="sensors/"/>
+  <xacro:property name="thruster_namespace" value="$(arg thruster_namespace)" scope="global" />
+  <xacro:property name="camera_namespace" value="$(arg camera_namespace)" scope="global" />
+  <xacro:property name="sensor_namespace" value="$(arg sensor_namespace)" scope="global" />
+  <xacro:property name="namespace" value="$(arg namespace)" scope="global" />
   <!-- Include macros for dynamics plugins -->
   <xacro:include filename="$(find ben_description)/urdf/ben_dynamics_plugin.xacro" />
   <!-- Attach hydrodynamics plugin -->
   <xacro:usv_dynamics_gazebo name="ben_dynamics_plugin" />
+  <xacro:include filename="$(find ben_description)/urdf/sensors/ben_gps.xacro" />
+  <xacro:ben_gps name="gps_ben" x="-0.85" />
+  <xacro:include filename="$(find ben_description)/urdf/sensors/ben_imu.xacro" />
+  <xacro:ben_imu name="imu_ben" y="-0.2" />
+  <xacro:include filename="$(find ben_description)/urdf/sensors/lidar.xacro" />
+  <xacro:lidar name="lidar_ben" y="-0.3" type="16_beam"/>
+  <xacro:include filename="$(find ben_description)/urdf/sensors/ben_camera.xacro" />
+  <xacro:ben_camera name="front_camera" y="0.3" x="0.75" P="${radians(15)}" />
   <!-- Robot mesh -->
   <xacro:include filename="$(find ben_description)/urdf/ben.urdf" />
-  <!-- Note: this is only used for some sensors that do not correctly use the
-  robotNamespace parameter -->
-  <xacro:arg name="namespace" default="ben"/>
-  <xacro:property name="namespace" value="$(arg namespace)" scope="global" />
   <!-- === Thruster === -->
-  <xacro:arg name="thruster_namespace" default="thrusters/"/>
-  <xacro:property name="thruster_namespace" value="$(arg thruster_namespace)" scope="global" />
   <xacro:include filename="$(find ben_description)/urdf/ben_thruster.xacro" />
 </robot>

Commit message: Progress towards a usable gazebo simulation of BEN.

File: urdf/ben.xacro (robot description, xacro)
@@ -4,5 +4,5 @@
   robotNamespace parameter -->
   <xacro:arg name="namespace" default="ben"/>
-  <xacro:arg name="thruster_namespace" default="thrusters/"/>
+  <xacro:arg name="thruster_namespace" default="thruster/"/>
   <xacro:arg name="camera_namespace" default="cameras/"/>
   <xacro:arg name="sensor_namespace" default="sensors/"/>
@@ -16,13 +16,13 @@
   <xacro:usv_dynamics_gazebo name="ben_dynamics_plugin" />
   <xacro:include filename="$(find ben_gazebo)/urdf/sensors/ben_gps.xacro" />
-  <xacro:ben_gps name="gps_ben" x="-0.85" />
+  <xacro:ben_gps name="gps_ben" />
   <xacro:include filename="$(find ben_gazebo)/urdf/sensors/ben_imu.xacro" />
-  <xacro:ben_imu name="imu_ben" y="-0.2" />
+  <xacro:ben_imu name="imu_ben" />
   <xacro:include filename="$(find ben_gazebo)/urdf/sensors/lidar.xacro" />
-  <xacro:lidar name="lidar_ben" y="-0.3" type="16_beam"/>
+  <xacro:lidar name="lidar_ben" x="-1.77" y="0.0" z="1.34" type="16_beam"/>
   <xacro:include filename="$(find ben_gazebo)/urdf/sensors/ben_camera.xacro" />
-  <xacro:ben_camera name="front_camera" y="0.3" x="0.75" P="${radians(15)}" />
+  <xacro:ben_camera name="front_camera" y="0.1" x="-1.307" z="0.742" P="${radians(0)}" />
   <!-- Robot mesh -->
-  <xacro:include filename="$(find ben_gazebo)/urdf/ben.urdf" />
+  <xacro:include filename="$(find ben_gazebo)/urdf/ben_mesh.xacro" />
   <!-- === Thruster === -->
   <xacro:include filename="$(find ben_gazebo)/urdf/ben_thruster.xacro" />

File: urdf/ben_dynamics_plugin.xacro (robot description, xacro)
@@ -5,5 +5,5 @@
     <gazebo>
       <plugin name="usv_dynamics_${name}" filename="libusv_gazebo_dynamics_plugin.so">
-        <bodyName>base_link</bodyName>
+        <bodyName>${namespace}/base_link</bodyName>
         <!-- Must be same as the ocean model!-->
         <waterLevel>0</waterLevel>

File: urdf/ben_thruster.xacro (robot description, xacro)
@@ -1,12 +1,12 @@
 <?xml version="1.0"?>
 <robot xmlns:xacro="http://ros.org/wiki/xacro">
-  <xacro:include filename="$(find wamv_description)/urdf/thrusters/engine.xacro" />
-  <xacro:engine prefix="center" position="-2.373776 0.0 0.318237" />
+  <xacro:include filename="$(find ben_gazebo)/urdf/jetdrive.xacro" />
+  <xacro:engine prefix="${namespace}/center" position="-2.15 0.0 -0.3" />
   <gazebo>
-    <plugin name="wamv_gazebo_thrust" filename="libusv_gazebo_thrust_plugin.so">
+    <plugin name="ben_gazebo_thrust" filename="libusv_gazebo_thrust_plugin.so">
       <cmdTimeout>1.0</cmdTimeout>
       <robotNamespace>${namespace}</robotNamespace>
-      <xacro:include filename="$(find wamv_gazebo)/urdf/thruster_layouts/wamv_gazebo_thruster_config.xacro" />
-      <xacro:wamv_gazebo_thruster_config name="center" />
+      <xacro:include filename="$(find ben_gazebo)/urdf/ben_gazebo_thruster_config.xacro" />
+      <xacro:ben_gazebo_thruster_config name="center" />
     </plugin>
   </gazebo>

File: urdf/sensors/ben_3d_lidar.xacro (robot description, xacro)
@@ -25,16 +25,10 @@
                                             x:=0.7 y:=0 z:=1.8
                                             R:=0 P:=0 Y:=0
-                                            post_Y:=0 post_z_from:=1.2965
                                             update_rate:=10 vertical_lasers:=16 samples:=1875 resolution:=0.1
                                             min_angle:=${-pi} max_angle:=${pi}
                                             min_vertical_angle:=${-pi/12} max_vertical_angle:=${pi/12}
                                             max_range:=130 noise_stddev:=0.01">
-    <!-- Define length variables for link positioning -->
-    <xacro:property name="platform_z" value="${post_z_from}"/>
-    <xacro:property name="post_to_post_arm_x" value="0.03"/>
-    <xacro:property name="post_arm_to_lidar_x" value="0.04"/>
-    <xacro:property name="post_arm_to_lidar_z" value="0.05"/>
     <!-- 3d lidar sensor -->
-    <link name="${name}_link">
+    <link name="${namespace}/${name}_link">
       <visual name="${name}_visual">
         <origin xyz="0 0 -0.035" rpy="0 0 0"/>
@@ -59,82 +53,11 @@
       </inertial>
     </link>
-    <!-- Define post length and mass based on desired z position of sensor -->
-    <xacro:property name="post_length" value="${z-platform_z-post_arm_to_lidar_z}"/>
-    <xacro:property name="post_mass_per_meter" value="0.9"/>
-    <xacro:property name="post_mass" value="${post_mass_per_meter * post_length}"/>
-    <xacro:property name="post_radius" value="0.0076"/>
-    <!-- Sensor post -->
-    <link name="${name}_post_link">
-      <visual>
-        <geometry>
-          <cylinder radius="${post_radius}" length="${post_length}"/>
-        </geometry>
-        <material name="${name}_post_material">
-          <color rgba="0.0 0.0 0.0 1.0"/>
-        </material>
-      </visual>
-      <collision name="${name}_post_collision">
-        <geometry>
-          <cylinder radius="${post_radius}" length="${post_length}"/>
-        </geometry>
-      </collision>
-      <inertial>
-        <mass value="${post_mass}"/>
-        <inertia
-          ixx="${(post_mass/12) * (3*post_radius*post_radius + post_length*post_length)}"
-          iyy="${(post_mass/12) * (3*post_radius*post_radius + post_length*post_length)}"
-          izz="${(post_mass/2) * (post_radius*post_radius)}"
-          ixy="0"
-          ixz="0"
-          iyz="0"/>
-      </inertial>
-    </link>
-    <!-- Sensor post arm -->
-    <link name="${name}_post_arm_link">
-      <visual name="${name}_post_arm_visual">
-        <origin xyz="-0.038 0 -0.003" rpy="${radians(-60)} 0 ${-pi/2}"/>
-        <geometry>
-          <mesh filename="package://vrx_gazebo/models/sensor_post/mesh/sensor_post_arm.dae"/>
-        </geometry>
-      </visual>
-      <collision name="${name}_post_arm_collision">
-        <origin xyz="0 0 0" rpy="${radians(-60)-pi/20} 0 ${-pi/2}"/>
-        <geometry>
-          <cylinder radius="0.008" length="0.065"/>
-        </geometry>
-      </collision>
-      <inertial>
-        <origin xyz="0 0 0" rpy="${radians(-60)-pi/20} 0 ${-pi/2}"/>
-        <mass value="0.1"/>
-        <inertia
-          ixx="0.00003680833"
-          iyy="0.00003680833"
-          izz="0.00000320000"
-          ixy="0"
-          ixz="0"
-          iyz="0"/>
-      </inertial>
-    </link>
-    <!-- Base to sensor post joint -->
-    <xacro:property name="post_z" value="${platform_z+post_length/2}"/>
-    <xacro:property name="post_to_lidar_x" value="${post_to_post_arm_x+post_arm_to_lidar_x}"/>
-    <joint name="base_to_${name}_post_joint" type="fixed">
-      <origin xyz="${x-(post_to_lidar_x)*cos(post_Y)} ${y-(post_to_lidar_x)*sin(post_Y)} ${post_z}" rpy="0 0 ${post_Y}" />
-      <parent link="base_link" />
-      <child link="${name}_post_link" />
+    <!-- Sensor post arm to lidar joint -->
+    <joint name="${namespace}/motion_sensor_to_${name}_joint" type="fixed">
+      <origin xyz="${x} ${y} ${z}" rpy="${R} ${P} ${Y}" />
+      <parent link="${namespace}/motion_sensor_link" />
+      <child link="${namespace}/${name}_link" />
     </joint>
-    <!-- Sensor post to sensor post arm joint -->
-    <joint name="${name}_post_to_${name}_post_arm_joint" type="fixed">
-      <origin xyz="${post_to_post_arm_x} 0 ${z-post_z-post_arm_to_lidar_z}" rpy="0 0 0" />
-      <parent link="${name}_post_link" />
-      <child link="${name}_post_arm_link" />
-    </joint>
-    <!-- Sensor post arm to lidar joint -->
-    <joint name="${name}_post_arm_to_${name}_joint" type="fixed">
-      <origin xyz="${post_arm_to_lidar_x} 0 ${post_arm_to_lidar_z}" rpy="${R} ${P} ${Y-post_Y}" />
-      <parent link="${name}_post_arm_link" />
-      <child link="${name}_link" />
-    </joint>
-    <gazebo reference="${name}_link">
+    <gazebo reference="${namespace}/${name}_link">
       <sensor type="gpu_ray" name="${name}_sensor">
         <update_rate>${update_rate}</update_rate>
@@ -171,8 +94,4 @@
       </sensor>
     </gazebo>
-    <!-- Set color of post -->
-    <gazebo reference="${name}_post_link">
-      <material>Gazebo/Black</material>
-    </gazebo>
   </xacro:macro>
 </robot>

File: urdf/sensors/ben_camera.xacro (robot description, xacro)
@@ -1,12 +1,7 @@
 <?xml version="1.0"?>
 <robot xmlns:xacro="http://ros.org/wiki/xacro">
-  <xacro:macro name="ben_camera" params="name x:=0.5 y:=0 z:=1.5 post_z_from:=1.2965 R:=0 P:=0 Y:=0 post_Y:=0">
-    <!-- Define length variables for link positioning -->
-    <xacro:property name="platform_z" value="${post_z_from}"/>
-    <xacro:property name="post_to_post_arm_x" value="0.03"/>
-    <xacro:property name="post_arm_to_camera_x" value="0.02"/>
-    <xacro:property name="post_arm_to_camera_z" value="0.027"/>
+  <xacro:macro name="ben_camera" params="name x:=0.5 y:=0 z:=1.5 R:=0 P:=0 Y:=0">
     <!-- Monocular Camera -->
-    <link name="${name}_link">
+    <link name="${namespace}/${name}_link">
       <visual name="${name}_visual">
         <origin xyz="-0.033 0 0" rpy="0 0 ${pi/2}"/>
@@ -41,92 +36,21 @@
     <!-- Define a link for the optical frame.  This will match the sensor frame and
          be oriented in the camera convention. -->
-    <link name="${name}_link_optical">
+    <link name="${namespace}/${name}_link_optical">
     </link>
-    <!-- Define post length and mass based on desired z position of sensor -->
-    <xacro:property name="post_length" value="${z-platform_z-post_arm_to_camera_z}"/>
-    <xacro:property name="post_mass_per_meter" value="0.9"/>
-    <xacro:property name="post_mass" value="${post_mass_per_meter * post_length}"/>
-    <xacro:property name="post_radius" value="0.0076"/>
-    <!-- Sensor post -->
-    <link name="${name}_post_link">
-      <visual>
-        <geometry>
-          <cylinder radius="${post_radius}" length="${post_length}"/>
-        </geometry>
-        <material name="${name}_post_material">
-          <color rgba="0.0 0.0 0.0 1.0"/>
-        </material>
-      </visual>
-      <collision name="${name}_post_collision">
-        <geometry>
-          <cylinder radius="${post_radius}" length="${post_length}"/>
-        </geometry>
-      </collision>
-      <inertial>
-        <mass value="${post_mass}"/>
-        <inertia
-          ixx="${(post_mass/12) * (3*post_radius*post_radius + post_length*post_length)}"
-          iyy="${(post_mass/12) * (3*post_radius*post_radius + post_length*post_length)}"
-          izz="${(post_mass/2) * (post_radius*post_radius)}"
-          ixy="0"
-          ixz="0"
-          iyz="0"/>
-      </inertial>
-    </link>
-    <!-- Sensor post arm -->
-    <link name="${name}_post_arm_link">
-      <visual name="${name}_post_arm_visual">
-        <origin xyz="-0.038 0 -0.003" rpy="${radians(-60)} 0 ${-pi/2}"/>
-        <geometry>
-          <mesh filename="package://vrx_gazebo/models/sensor_post/mesh/sensor_post_arm.dae"/>
-        </geometry>
-      </visual>
-      <collision name="${name}_post_arm_collision">
-        <origin xyz="0 0 0" rpy="${radians(-60)-pi/20} 0 ${-pi/2}"/>
-        <geometry>
-          <cylinder radius="0.008" length="0.065"/>
-        </geometry>
-      </collision>
-      <inertial>
-        <origin xyz="0 0 0" rpy="${radians(-60)-pi/20} 0 ${-pi/2}"/>
-        <mass value="0.1"/>
-        <inertia
-          ixx="0.00003680833"
-          iyy="0.00003680833"
-          izz="0.00000320000"
-          ixy="0"
-          ixz="0"
-          iyz="0"/>
-      </inertial>
-    </link>
-    <!-- Base to sensor post joint -->
-    <xacro:property name="post_z" value="${platform_z+post_length/2}"/>
-    <xacro:property name="post_to_camera_x" value="${post_to_post_arm_x+post_arm_to_camera_x}"/>
-    <joint name="base_to_${name}_post_joint" type="fixed">
-      <origin xyz="${x-(post_to_camera_x)*cos(post_Y)} ${y-(post_to_camera_x)*sin(post_Y)} ${post_z}" rpy="0 0 ${post_Y}" />
-      <parent link="base_link" />
-      <child link="${name}_post_link" />
-    </joint>
-    <!-- Sensor post to sensor post arm joint -->
-    <joint name="${name}_post_to_${name}_post_arm_joint" type="fixed">
-      <origin xyz="${post_to_post_arm_x} 0 ${z-post_z-post_arm_to_camera_z}" rpy="0 0 0" />
-      <parent link="${name}_post_link" />
-      <child link="${name}_post_arm_link" />
-    </joint>
     <!-- Sensor post arm to camera joint -->
-    <joint name="${name}_post_arm_to_${name}_joint" type="fixed">
-      <origin xyz="${post_arm_to_camera_x} 0 ${post_arm_to_camera_z}" rpy="${R} ${P} ${Y-post_Y}" />
-      <parent link="${name}_post_arm_link" />
-      <child link="${name}_link" />
+    <joint name="${namespace}/motion_sensor_to_${name}_joint" type="fixed">
+      <origin xyz="${x} ${y} ${z}" rpy="${R} ${P} ${Y}" />
+      <parent link="${namespace}/motion_sensor_link" />
+      <child link="${namespace}/${name}_link" />
     </joint>
     <!-- Camera to optical frame joint.  This is oriented to convert between ENU
          and camera conventions -->
-    <joint name="${name}_to_${name}_link_optical_joint" type="fixed">
+    <joint name="${namespace}/${name}_to_${name}_link_optical_joint" type="fixed">
       <origin xyz="0 0 0" rpy="${-pi/2} 0 ${-pi/2}" />
-      <parent link="${name}_link" />
-      <child link="${name}_link_optical" />
+      <parent link="${namespace}/${name}_link" />
+      <child link="${namespace}/${name}_link_optical" />
     </joint>
     <!-- Gazebo camera setup -->
-    <gazebo reference="${name}_link">
+    <gazebo reference="${namespace}/${name}_link">
       <sensor type="camera" name="${name}_sensor">
         <update_rate>30.0</update_rate>
@@ -167,8 +91,4 @@
       </sensor>
     </gazebo>
-    <!-- Set color of post -->
-    <gazebo reference="${name}_post_link">
-      <material>Gazebo/Black</material>
-    </gazebo>
   </xacro:macro>
 </robot>

File: urdf/sensors/ben_gps.xacro (robot description, xacro)
@@ -1,23 +1,6 @@
 <?xml version="1.0" encoding="UTF-8"?>
 <robot xmlns:xacro="http://ros.org/wiki/xacro">
-  <xacro:macro name="ben_gps" params="name:=gps x:=0.3 y:=0 z:=1.3 R:=0 P:=0 Y:=0 lat:=21.30996 lon:=-157.8901 elev:=0.0 update_rate:=15">
-    <link name="${name}_link">
-      <visual name="${name}_visual">
-        <geometry>
-          <mesh filename="package://wamv_gazebo/models/gps/mesh/gps.dae"/>
-        </geometry>
-      </visual>
-      <collision name="${name}_collision_base">
-        <origin xyz="0 0 0.025" rpy="0 0 0" />
-        <geometry>
-          <cylinder length="0.05" radius="0.015" />
-        </geometry>
-      </collision>
-      <collision name="${name}_collision_antenna">
-        <origin xyz="0 0 0.11" rpy="0 0 0" />
-        <geometry>
-          <cylinder length="0.1" radius="0.15" />
-        </geometry>
-      </collision>
+  <xacro:macro name="ben_gps" params="name:=gps update_rate:=15">
+    <link name="${namespace}/${name}_link">
       <inertial>
         <mass value="1"/>
@@ -25,10 +8,9 @@
       </inertial>
     </link>
-    <joint name="${name}_joint" type="revolute">
+    <joint name="${namespace}/${name}_joint" type="revolute">
       <axis xyz="0 0 1"/>
       <limit effort="1000.0" lower="0.0" upper="0" velocity="0"/>
-      <origin xyz="${x} ${y} ${z}" rpy="${R} ${P} ${Y}" />
-      <parent link="base_link" />
-      <child link="${name}_link" />
+      <parent link="${namespace}/motion_sensor_link" />
+      <child link="${namespace}/${name}_link" />
     </joint>
     <gazebo>
@@ -36,5 +18,5 @@
         <updateRate>${update_rate}</updateRate>
         <alwaysOn>true</alwaysOn>
-        <bodyName>${name}_link</bodyName>
+        <bodyName>${namespace}/${name}_link</bodyName>
         <!-- Manually prepend namespace to tf frame. -->
         <frameId>${namespace}/${name}_link</frameId>
@@ -46,9 +28,5 @@
              https://bitbucket.org/osrf/vrx/issues/64 -->
         <velocityTopicName>${namespace}/${sensor_namespace}gps/gps/fix_velocity</velocityTopicName>
-        <!-- Location of origin of Gazebo Sand Island map -->
-        <referenceLatitude>${lat}</referenceLatitude>
-        <referenceLongitude>${lon}</referenceLongitude>
-        <referenceAltitude>${elev}</referenceAltitude>
-        <referenceHeading>90</referenceHeading>
+        <useWorldSphericalCoordinates>true</useWorldSphericalCoordinates>
         <offset>0.0 0.0 0.0</offset>
         <drift>0.0 0.0 0.0</drift>

File: urdf/sensors/ben_imu.xacro (robot description, xacro)
@@ -1,14 +1,6 @@
 <?xml version="1.0"?>
 <robot xmlns:xacro="http://ros.org/wiki/xacro">
-  <xacro:macro name="ben_imu" params="name:=imu x:=0.3 y:=0.5 z:=1.3 R:=0 P:=0 Y:=0 update_rate:=15">
-    <link name="${name}_link">
-      <visual name="${name}_visual">>
-        <geometry>
-          <box size="0.05 0.025 0.005" />
-        </geometry>
-        <material name="${name}_visual_material">
-          <color rgba="1.0 0.0 00 1.0" />
-        </material>
-      </visual>
+  <xacro:macro name="ben_imu" params="name:=imu update_rate:=15">
+    <link name="${namespace}/${name}_link">
       <inertial>
         <mass value="0.1"/>
@@ -16,15 +8,14 @@
       </inertial>
     </link>
-    <joint name="${name}_joint" type="revolute">
+    <joint name="${namespace}/${name}_joint" type="revolute">
       <axis xyz="0 0 1"/>
       <limit effort="1000.0" lower="0.0" upper="0" velocity="0"/>
-      <origin xyz="${x} ${y} ${z}" rpy="${R} ${P} ${Y}"/>
-      <parent link="base_link"/>
-      <child link="${name}_link"/>
+      <parent link="${namespace}/motion_sensor_link"/>
+      <child link="${namespace}/${name}_link"/>
     </joint>
     <gazebo>
       <plugin name="imu_plugin_${name}" filename="libhector_gazebo_ros_imu.so">
         <updateRate>${update_rate}</updateRate>
-        <bodyName>${name}_link</bodyName>
+        <bodyName>${namespace}/${name}_link</bodyName>
         <topicName>${namespace}/${sensor_namespace}imu/imu/data</topicName>
         <serviceName>${namespace}/${sensor_namespace}imu_service</serviceName>

File: urdf/sensors/lidar.xacro (robot description, xacro)
@@ -6,11 +6,9 @@
                          name
                          x:=0.7 y:=0 z:=1.8
-                         R:=0 P:=0 Y:=0
-                         post_Y:=0 post_z_from:=1.2965">
+                         R:=0 P:=0 Y:=0">
     <xacro:if value="${type == '16_beam'}">
       <xacro:ben_3d_lidar name="${name}"
                            x="${x}" y="${y}" z="${z}"
                            R="${R}" P="${P}" Y="${Y}"
-                           post_Y="${post_Y}" post_z_from="${post_z_from}"
                            vertical_lasers="16"/>
       <!--specs for 16 beam lidar are implemented by default.
@@ -21,5 +19,4 @@
                            x="${x}" y="${y}" z="${z}"
                            R="${R}" P="${P}" Y="${Y}"
-                           post_Y="${post_Y}" post_z_from="${post_z_from}"
                            vertical_lasers="32"
                            samples="2187"
