Commit message: Add camera array, posmv, factory gps

File: urdf/ben.xacro (robot description, xacro)
@@ -15,12 +15,16 @@
   <!-- Attach hydrodynamics plugin -->
   <xacro:usv_dynamics_gazebo name="ben_dynamics_plugin" />
-  <xacro:include filename="$(find ben_gazebo)/urdf/sensors/ben_gps.xacro" />
-  <xacro:ben_gps name="gps_ben" />
-  <xacro:include filename="$(find ben_gazebo)/urdf/sensors/ben_imu.xacro" />
-  <xacro:ben_imu name="imu_ben" />
+  <xacro:include filename="$(find ben_gazebo)/urdf/sensors/ben_factory_gps.xacro" />
+  <xacro:ben_factory_gps name="gps_ben" />
+  <xacro:include filename="$(find ben_gazebo)/urdf/sensors/ben_factory_heading_sensor.xacro" />
+  <xacro:ben_factory_heading_sensor name="heading_ben" />
+  <xacro:include filename="$(find ben_gazebo)/urdf/sensors/ben_posmv.xacro" />
+  <xacro:ben_posmv name="posmv_ben" />
   <xacro:include filename="$(find ben_gazebo)/urdf/sensors/lidar.xacro" />
   <xacro:lidar name="lidar_ben" x="-1.77" y="0.0" z="1.34" type="16_beam"/>
   <xacro:include filename="$(find ben_gazebo)/urdf/sensors/ben_camera.xacro" />
   <xacro:ben_camera name="front_camera" y="0.1" x="-1.307" z="0.742" P="${radians(0)}" />
+  <xacro:include filename="$(find ben_gazebo)/urdf/sensors/ben_pano_array.xacro" />
+  <xacro:ben_pano_array name="pano" y="0.0" x="0.0" z="1.0"/>
   <!-- Robot mesh -->
   <xacro:include filename="$(find ben_gazebo)/urdf/ben_mesh.xacro" />

File: urdf/ben_gazebo_thruster_config.xacro (robot description, xacro)
@@ -1,12 +1,12 @@
 <?xml version="1.0"?>
 <plugin xmlns:xacro="http://ros.org/wiki/xacro">
-  <xacro:macro  name="ben_gazebo_thruster_config" params="name enable_angle:=true">
+  <xacro:macro  name="ben_gazebo_thruster_config" params="enable_angle:=true">
     <thruster>
       <!-- Required Parameters -->
-      <linkName>${namespace}/${name}_propeller_link</linkName>
-      <propJointName>${namespace}/${name}_engine_propeller_joint</propJointName>
-      <engineJointName>${namespace}/${name}_chasis_engine_joint</engineJointName>
-      <cmdTopic>${thruster_namespace}${name}_thrust_cmd</cmdTopic>
-      <angleTopic>${thruster_namespace}${name}_thrust_angle</angleTopic>
+      <linkName>${namespace}/propeller_link</linkName>
+      <propJointName>${namespace}/engine_propeller_joint</propJointName>
+      <engineJointName>${namespace}/chasis_engine_joint</engineJointName>
+      <cmdTopic>${thruster_namespace}thrust_cmd</cmdTopic>
+      <angleTopic>${thruster_namespace}thrust_angle</angleTopic>
       <enableAngle>${enable_angle}</enableAngle>
       <!-- Optional Parameters -->

File: urdf/ben_thruster.xacro (robot description, xacro)
@@ -2,5 +2,5 @@
 <robot xmlns:xacro="http://ros.org/wiki/xacro">
   <xacro:include filename="$(find ben_gazebo)/urdf/jetdrive.xacro" />
-  <xacro:engine prefix="${namespace}/center" position="-2.15 0.0 -0.3" />
+  <xacro:engine prefix="${namespace}/" position="-2.15 0.0 -0.3" />
   <gazebo>
     <plugin name="ben_gazebo_thrust" filename="libusv_gazebo_thrust_plugin.so">
@@ -8,5 +8,5 @@
       <robotNamespace>${namespace}</robotNamespace>
       <xacro:include filename="$(find ben_gazebo)/urdf/ben_gazebo_thruster_config.xacro" />
-      <xacro:ben_gazebo_thruster_config name="center" />
+      <xacro:ben_gazebo_thruster_config/>
     </plugin>
   </gazebo>

File: urdf/jetdrive.xacro (robot description, xacro)
@@ -3,5 +3,5 @@
   <!-- Macro for inserting an engine with its propeller. -->
   <xacro:macro name="engine" params="prefix position:='0 0 0' orientation:='0 0 0'">
-    <link name="${prefix}_engine_link">
+    <link name="${prefix}engine_link">
       <visual>
         <geometry>
@@ -9,5 +9,5 @@
         </geometry>
       </visual>
-      <collision name="${prefix}_engine_vertical_axis_collision">
+      <collision name="${prefix}engine_vertical_axis_collision">
         <origin xyz="-0.16 0 -0.24" rpy="0 0 0" />
         <geometry>
@@ -15,5 +15,5 @@
         </geometry>
       </collision>
-      <collision name="${prefix}_engine_rear_end_collision">
+      <collision name="${prefix}engine_rear_end_collision">
         <origin xyz="-0.34 0 0.12" rpy="0 0 0" />
         <geometry>
@@ -26,5 +26,5 @@
       </inertial>
     </link>
-    <link name="${prefix}_propeller_link">
+    <link name="${prefix}propeller_link">
       <visual>
         <geometry>
@@ -32,5 +32,5 @@
         </geometry>
       </visual>
-      <collision name="${prefix}_propeller_collision">
+      <collision name="${prefix}propeller_collision">
         <origin xyz="-0.08 0 0" rpy="0 1.57 0" />
         <geometry>
@@ -43,15 +43,15 @@
       </inertial>
     </link>
-    <joint name="${prefix}_chasis_engine_joint" type="revolute">
+    <joint name="${prefix}chasis_engine_joint" type="revolute">
       <axis xyz="0 0 1"/>
       <limit lower="${-pi}" upper="${pi}" effort="10" velocity="10"/>
       <origin xyz="${position}" rpy="${orientation}"/>
       <parent link="${namespace}/motion_sensor_link"/>
-      <child link="${prefix}_engine_link"/>
+      <child link="${prefix}engine_link"/>
     </joint>
-    <joint name="${prefix}_engine_propeller_joint" type="continuous">
+    <joint name="${prefix}engine_propeller_joint" type="continuous">
       <axis rpy="0 0 0" xyz="1 0 0"/>
-      <parent link="${prefix}_engine_link"/>
-      <child link="${prefix}_propeller_link"/>
+      <parent link="${prefix}engine_link"/>
+      <child link="${prefix}propeller_link"/>
       <origin rpy="0 0 0" xyz="-0.278156 0 -0.509371"/>
       <limit effort="100" velocity="100" />

File: urdf/sensors/ben_factory_gps.xacro (robot description, xacro)
@@ -1,5 +1,5 @@
 <?xml version="1.0" encoding="UTF-8"?>
 <robot xmlns:xacro="http://ros.org/wiki/xacro">
-  <xacro:macro name="ben_gps" params="name:=gps update_rate:=15">
+  <xacro:macro name="ben_factory_gps" params="name:=gps update_rate:=5">
     <link name="${namespace}/${name}_link">
       <inertial>
@@ -13,4 +13,5 @@
       <parent link="${namespace}/motion_sensor_link" />
       <child link="${namespace}/${name}_link" />
+      <origin xyz="-0.953 0.103 0.628" rpy="0 0 0"/>
     </joint>
     <gazebo>
@@ -21,5 +22,5 @@
         <!-- Manually prepend namespace to tf frame. -->
         <frameId>${namespace}/${name}_link</frameId>
-        <topicName>${namespace}/${sensor_namespace}gps/fix</topicName>
+        <topicName>${namespace}/${sensor_namespace}gps/position</topicName>
         <!-- Note that the hector_gazebo_ros_gps plugin uses NWU coordinates
              for reporting velocities.  This may cause problems if localization
@@ -27,9 +28,10 @@
              See Issue #64 in VRX project for details
              https://bitbucket.org/osrf/vrx/issues/64 -->
-        <velocityTopicName>${namespace}/${sensor_namespace}gps/fix_velocity</velocityTopicName>
+        <velocityTopicName>${namespace}/${sensor_namespace}gps/velocity</velocityTopicName>
         <useWorldSphericalCoordinates>true</useWorldSphericalCoordinates>
         <offset>0.0 0.0 0.0</offset>
-        <drift>0.0 0.0 0.0</drift>
-        <gaussianNoise>0 0 0</gaussianNoise>
+        <drift>0.5 0.5 0.5</drift>
+        <driftFrequency>0.1 0.1 0.1</driftFrequency>
+        <gaussianNoise>0.1 0.1 0.1</gaussianNoise>
         <velocityOffset>0.0 0.0 0.0</velocityOffset>
         <velocityDrift>0.0 0.0 0.0</velocityDrift>

File: urdf/sensors/ben_factory_heading_sensor.xacro (robot description, xacro)
@@ -1,5 +1,5 @@
 <?xml version="1.0"?>
 <robot xmlns:xacro="http://ros.org/wiki/xacro">
-  <xacro:macro name="ben_imu" params="name:=imu update_rate:=15">
+  <xacro:macro name="ben_factory_heading_sensor" params="name:=heading update_rate:=5">
     <link name="${namespace}/${name}_link">
       <inertial>
@@ -18,13 +18,13 @@
         <updateRate>${update_rate}</updateRate>
         <bodyName>${namespace}/${name}_link</bodyName>
-        <topicName>${namespace}/${sensor_namespace}imu/data</topicName>
-        <serviceName>${namespace}/${sensor_namespace}imu_service</serviceName>
+        <topicName>${namespace}/${sensor_namespace}heading</topicName>
+        <serviceName>${namespace}/${sensor_namespace}heading_service</serviceName>
         <!-- Manually prepend namespace to tf frame. -->
         <frameId>${namespace}/${name}_link</frameId>
         <alwaysOn>true</alwaysOn>
         <accelOffset>0.0 0.0 0.0</accelOffset>
-        <accelDrift>0.0 0.0 0.0</accelDrift>
+        <accelDrift>3.14 3.14 0.001</accelDrift>
         <accelDriftFrequency>0.00027 0.00027 0.000027</accelDriftFrequency>
-        <accelGaussianNoise>0.0 0.0 0.0</accelGaussianNoise>
+        <accelGaussianNoise>1.0 1.0 0.001</accelGaussianNoise>
         <rateOffset>0.0 0.0 0.0</rateOffset>
         <rateDrift>0.0 0.0 0.0</rateDrift>

File: urdf/sensors/ben_posmv.xacro (robot description, xacro)
@@ -1,5 +1,5 @@
 <?xml version="1.0" encoding="UTF-8"?>
 <robot xmlns:xacro="http://ros.org/wiki/xacro">
-  <xacro:macro name="ben_gps" params="name:=gps update_rate:=15">
+  <xacro:macro name="ben_posmv" params="name:=posmv update_rate:=100">
     <link name="${namespace}/${name}_link">
       <inertial>
@@ -15,5 +15,5 @@
     </joint>
     <gazebo>
-      <plugin name="gps_plugin_${name}" filename="libhector_gazebo_ros_gps.so">
+      <plugin name="posmv_gps_plugin_${name}" filename="libhector_gazebo_ros_gps.so">
         <updateRate>${update_rate}</updateRate>
         <alwaysOn>true</alwaysOn>
@@ -21,5 +21,5 @@
         <!-- Manually prepend namespace to tf frame. -->
         <frameId>${namespace}/${name}_link</frameId>
-        <topicName>${namespace}/${sensor_namespace}gps/fix</topicName>
+        <topicName>${namespace}/${sensor_namespace}posmv/position</topicName>
         <!-- Note that the hector_gazebo_ros_gps plugin uses NWU coordinates
              for reporting velocities.  This may cause problems if localization
@@ -27,5 +27,5 @@
              See Issue #64 in VRX project for details
              https://bitbucket.org/osrf/vrx/issues/64 -->
-        <velocityTopicName>${namespace}/${sensor_namespace}gps/fix_velocity</velocityTopicName>
+        <velocityTopicName>${namespace}/${sensor_namespace}posmv/velocity</velocityTopicName>
         <useWorldSphericalCoordinates>true</useWorldSphericalCoordinates>
         <offset>0.0 0.0 0.0</offset>
@@ -36,4 +36,25 @@
         <velocityGaussianNoise>0.0 0.0 0.0</velocityGaussianNoise>
       </plugin>
+      <plugin name="posmv_imu_plugin_${name}" filename="libhector_gazebo_ros_imu.so">
+        <updateRate>${update_rate}</updateRate>
+        <bodyName>${namespace}/${name}_link</bodyName>
+        <topicName>${namespace}/${sensor_namespace}posmv/orientation</topicName>
+        <serviceName>${namespace}/${sensor_namespace}posmv/imu_service</serviceName>
+        <!-- Manually prepend namespace to tf frame. -->
+        <frameId>${namespace}/${name}_link</frameId>
+        <alwaysOn>true</alwaysOn>
+        <accelOffset>0.0 0.0 0.0</accelOffset>
+        <accelDrift>0.0 0.0 0.0</accelDrift>
+        <accelDriftFrequency>0.00027 0.00027 0.000027</accelDriftFrequency>
+        <accelGaussianNoise>0.0 0.0 0.0</accelGaussianNoise>
+        <rateOffset>0.0 0.0 0.0</rateOffset>
+        <rateDrift>0.0 0.0 0.0</rateDrift>
+        <rateDriftFrequency>0.00027 0.00027 0.000027</rateDriftFrequency>
+        <rateGaussianNoise>0.0 0.0 0.0</rateGaussianNoise>
+        <yawOffset>0.0</yawOffset>
+        <yawDrift>0.0</yawDrift>
+        <yawDriftFrequency>0.00027</yawDriftFrequency>
+        <yawGaussianNoise>0.0</yawGaussianNoise>
+      </plugin>
     </gazebo>
   </xacro:macro>

Commit message: Switch to new mru plugin for posmv and gps from gazebo

File: urdf/ben.xacro (robot description, xacro)
@@ -19,6 +19,6 @@
   <xacro:include filename="$(find ben_gazebo)/urdf/sensors/ben_factory_heading_sensor.xacro" />
   <xacro:ben_factory_heading_sensor name="heading_ben" />
-  <xacro:include filename="$(find ben_gazebo)/urdf/sensors/ben_posmv.xacro" />
-  <xacro:ben_posmv name="posmv_ben" />
+  <xacro:include filename="$(find ben_gazebo)/urdf/sensors/ben_posmv_mru.xacro" />
+  <xacro:ben_posmv/>
   <xacro:include filename="$(find ben_gazebo)/urdf/sensors/lidar.xacro" />
   <xacro:lidar name="lidar_ben" x="-1.77" y="0.0" z="1.34" type="16_beam"/>
@@ -26,5 +26,5 @@
   <xacro:ben_camera name="front_camera" y="0.1" x="-1.307" z="0.742" P="${radians(0)}" />
   <xacro:include filename="$(find ben_gazebo)/urdf/sensors/ben_pano_array.xacro" />
-  <xacro:ben_pano_array name="pano" y="0.0" x="0.0" z="1.0"/>
+  <xacro:ben_pano_array name="pano" x="-1.77" z="1.4"/>
   <!-- Robot mesh -->
   <xacro:include filename="$(find ben_gazebo)/urdf/ben_mesh.xacro" />

File: urdf/sensors/ben_factory_gps.xacro (robot description, xacro)
@@ -2,5 +2,5 @@
 <robot xmlns:xacro="http://ros.org/wiki/xacro">
   <xacro:macro name="ben_factory_gps" params="name:=gps update_rate:=5">
-    <link name="${namespace}/${name}_link">
+    <link name="${namespace}/${name}">
       <inertial>
         <mass value="1"/>
@@ -12,30 +12,55 @@
       <limit effort="1000.0" lower="0.0" upper="0" velocity="0"/>
       <parent link="${namespace}/motion_sensor_link" />
-      <child link="${namespace}/${name}_link" />
+      <child link="${namespace}/${name}" />
       <origin xyz="-0.953 0.103 0.628" rpy="0 0 0"/>
     </joint>
     <gazebo>
-      <plugin name="gps_plugin_${name}" filename="libhector_gazebo_ros_gps.so">
+      <sensor type="gps" name="${namespace}/${name}_gps">
+        <plugin name="gps_plugin_${name}" filename="libgazebo_ros_mru.so">
+          <positionTopic>${namespace}/${sensor_namespace}gps/position</positionTopic>
+          <velocityTopic>${namespace}/${sensor_namespace}gps/velocity</velocityTopic>
+          <frameId>${namespace}/${name}</frameId>
+        </plugin>
         <updateRate>${update_rate}</updateRate>
         <alwaysOn>true</alwaysOn>
-        <bodyName>${namespace}/${name}_link</bodyName>
-        <!-- Manually prepend namespace to tf frame. -->
-        <frameId>${namespace}/${name}_link</frameId>
-        <topicName>${namespace}/${sensor_namespace}gps/position</topicName>
-        <!-- Note that the hector_gazebo_ros_gps plugin uses NWU coordinates
-             for reporting velocities.  This may cause problems if localization
-             requires velocity in ENU.
-             See Issue #64 in VRX project for details
-             https://bitbucket.org/osrf/vrx/issues/64 -->
-        <velocityTopicName>${namespace}/${sensor_namespace}gps/velocity</velocityTopicName>
-        <useWorldSphericalCoordinates>true</useWorldSphericalCoordinates>
-        <offset>0.0 0.0 0.0</offset>
-        <drift>0.5 0.5 0.5</drift>
-        <driftFrequency>0.1 0.1 0.1</driftFrequency>
-        <gaussianNoise>0.1 0.1 0.1</gaussianNoise>
-        <velocityOffset>0.0 0.0 0.0</velocityOffset>
-        <velocityDrift>0.0 0.0 0.0</velocityDrift>
-        <velocityGaussianNoise>0.0 0.0 0.0</velocityGaussianNoise>
-      </plugin>
+        <gps>
+          <position_sensing>
+            <horizontal>
+              <noise type="gaussian">
+                <mean>0.0</mean>
+                <stddev>1.7e-2</stddev>
+                <bias_mean>0.5</bias_mean>
+                <bias_stddev>0.01</bias_stddev>
+              </noise>
+            </horizontal>
+            <vertical>
+              <noise type="gaussian">
+                <mean>0.0</mean>
+                <stddev>1.7e-2</stddev>
+                <bias_mean>0.75</bias_mean>
+                <bias_stddev>0.01</bias_stddev>
+              </noise>
+            </vertical>
+          </position_sensing>
+          <velocity_sensing>
+            <horizontal>
+              <noise type="gaussian">
+                <mean>0.0</mean>
+                <stddev>1.7e-2</stddev>
+                <bias_mean>0.1</bias_mean>
+                <bias_stddev>0.001</bias_stddev>
+              </noise>
+            </horizontal>
+            <vertical>
+              <noise type="gaussian">
+                <mean>0.0</mean>
+                <stddev>1.7e-2</stddev>
+                <bias_mean>0.1</bias_mean>
+                <bias_stddev>0.001</bias_stddev>
+              </noise>
+            </vertical>
+          </velocity_sensing>
+        </gps>
+      </sensor>
     </gazebo>
   </xacro:macro>

File: urdf/sensors/ben_pano_array.xacro (robot description, xacro)
@@ -6,9 +6,12 @@
         <origin xyz="0 0 0" rpy="0 0 0"/>
         <geometry>
-          <cylinder radius="0.05" length="0.05"/>
+          <mesh filename="package://ben_gazebo/models/meshes/panoramic_camera_housing.dae"/>
         </geometry>
       </visual>
       <collision name="${name}_collision">
-          <cylinder radius="0.05" length="0.05"/>
+        <origin xyz="0 0 0.05" rpy="0 0 0"/>
+        <geometry>
+          <cylinder radius="0.15" length="0.1"/>
+        </geometry>
       </collision>
       <!-- Model inertia as box with <size>0.078 0.03 0.03</size> -->
@@ -31,5 +34,5 @@
     <xacro:include filename="$(find ben_gazebo)/urdf/sensors/ben_pano_camera.xacro" />
     <xacro:macro name="loop" params="i">
-      <xacro:ben_pano_camera name="${name}" number="${i}" x="0.1" Y="${-radians(i*60)}" />
+      <xacro:ben_pano_camera name="${name}" number="${i}" x="0.08" z="0.05" Y="${-radians(i*60)}" />
       <xacro:if value="${i}">
         <xacro:loop i="${i-1}" />

File: urdf/sensors/ben_pano_camera.xacro (robot description, xacro)
@@ -55,7 +55,15 @@
          and camera conventions -->
     <joint name="${namespace}/${name}_${number}_to_${name}_${number}_optical_joint" type="fixed">
-      <origin xyz="10 0 0" rpy="${-pi/2} 0 ${-pi/2}" />
+      <origin xyz="0 0 0" rpy="${-pi/2} 0 ${-pi/2}" />
       <parent link="${namespace}/${name}_${number}" />
       <child link="${namespace}/${name}_${number}_optical" />
+    </joint>
+    <!--Move a reference plane away from the camera to project on in rviz-->
+    <link name="${namespace}/${name}_${number}_optical_rviz_mesh">
+    </link>
+    <joint name="${namespace}/${name}_${number}_optical_to_${name}_${number}_optical_rviz_mesh_joint" type="fixed">
+      <origin xyz="0 0 10" rpy="0 0 0" />
+      <parent link="${namespace}/${name}_${number}_optical" />
+      <child link="${namespace}/${name}_${number}_optical_rviz_mesh" />
     </joint>
     <!-- Gazebo camera setup -->
