Commit message: Split the gazebo parts away into a different package

File: urdf/ben_mesh.xacro (robot description, xacro)
@@ -1,4 +1,6 @@
 <?xml version="1.0"?>
 <robot xmlns:xacro="http://ros.org/wiki/xacro" name="ben">
+  <xacro:arg name="namespace" default="ben"/>
+  <xacro:property name="namespace" value="$(arg namespace)" scope="global" />
   <xacro:property name="mass" value="950" />
   <xacro:property name="cg_x" value="-0.911" />
@@ -16,16 +18,16 @@
   <joint name="${namespace}_base_to_motion_sensor_joint" type="fixed">
       <parent link="${namespace}/base_link"/>
-      <child link="${namespace}/motion_sensor_link"/>
+      <child link="${namespace}/motion_sensor"/>
       <origin xyz="${- cg_x} ${- cg_y} ${buoyancy_offset - cg_z}" rpy="0 0 0"/>
   </joint>
-  <link name="${namespace}/motion_sensor_link">
+  <link name="${namespace}/motion_sensor">
     <visual>
         <geometry>
-            <mesh filename="package://ben_gazebo/models/meshes/BEN_shell.dae"/>
+            <mesh filename="package://ben_description/models/meshes/BEN_shell.dae"/>
         </geometry>
     </visual>
     <collision>
         <geometry>
-            <mesh filename="package://ben_gazebo/models/meshes/BEN_convex_hull.dae"/>
+            <mesh filename="package://ben_description/models/meshes/BEN_convex_hull.dae"/>
         </geometry>
     </collision>
@@ -40,3 +42,13 @@
     </inertial>
   </link>
+  <xacro:include filename="$(find ben_description)/urdf/sensors/lidar.xacro" />
+  <xacro:ben_lidar name="lidar" x="-1.77" y="0.0" z="1.38"/>
+  <xacro:include filename="$(find ben_description)/urdf/sensors/pano_array.xacro" />
+  <xacro:pano_array name="pano" x="-1.77" z="1.42"/>
+  <xacro:include filename="$(find ben_description)/urdf/sensors/oem_gps.xacro" />
+  <xacro:oem_gps name="gps" x="-0.953" y="0.103" z="0.628"/>
+  <xacro:include filename="$(find ben_description)/urdf/sensors/oem_heading_sensor.xacro" />
+  <xacro:oem_heading_sensor name="heading"/>
+  <xacro:include filename="$(find ben_description)/urdf/sensors/forward_camera.xacro" />
+  <xacro:forward_camera name="forward_camera" y="0.1" x="-1.307" z="0.742" P="${radians(0)}" />
 </robot>

File: urdf/jetdrive.xacro (robot description, xacro)
@@ -47,5 +47,5 @@
       <limit lower="${-pi}" upper="${pi}" effort="10" velocity="10"/>
       <origin xyz="${position}" rpy="${orientation}"/>
-      <parent link="${namespace}/motion_sensor_link"/>
+      <parent link="${namespace}/motion_sensor"/>
       <child link="${prefix}engine_link"/>
     </joint>

File: urdf/sensors/lidar.xacro (robot description, xacro)
@@ -1,27 +1,35 @@
 <?xml version="1.0" encoding="UTF-8"?>
 <robot xmlns:xacro="http://ros.org/wiki/xacro">
-  <xacro:include filename="$(find ben_gazebo)/urdf/sensors/ben_3d_lidar.xacro"/>
-  <xacro:macro name="lidar"
-               params = "type:='16_beam'
-                         name
-                         x:=0.7 y:=0 z:=1.8
-                         R:=0 P:=0 Y:=0">
-    <xacro:if value="${type == '16_beam'}">
-      <xacro:ben_3d_lidar name="${name}"
-                           x="${x}" y="${y}" z="${z}"
-                           R="${R}" P="${P}" Y="${Y}"
-                           vertical_lasers="16"/>
-      <!--specs for 16 beam lidar are implemented by default.
-          See wamv_3d_lidar for those-->
-    </xacro:if>
-    <xacro:if value="${type == '32_beam'}">
-      <xacro:ben_3d_lidar name="${name}"
-                           x="${x}" y="${y}" z="${z}"
-                           R="${R}" P="${P}" Y="${Y}"
-                           vertical_lasers="32"
-                           samples="2187"
-                           min_vertical_angle="-0.186"
-                           max_vertical_angle="0.54"/>
-    </xacro:if>
+  <xacro:macro name="ben_lidar" params="name
+                                        x:=0.7 y:=0 z:=1.8
+                                        R:=0 P:=0 Y:=0">
+    <link name="${namespace}/${name}">
+      <visual name="${name}_visual">
+        <origin xyz="0 0 0" rpy="0 0 0"/>
+        <geometry>
+          <cylinder radius="0.055" length="0.075"/>
+        </geometry>
+      </visual>
+      <collision name="${name}_collision">
+        <geometry>
+          <cylinder radius="0.055" length="0.075"/>
+        </geometry>
+      </collision>
+      <inertial>
+        <mass value="1"/>
+        <inertia
+          ixx="0.00109375"
+          iyy="0.00109375"
+          izz="0.00125"
+          ixy="0"
+          ixz="0"
+          iyz="0"/>
+      </inertial>
+    </link>
+    <joint name="${namespace}/motion_sensor_to_${name}_joint" type="fixed">
+      <origin xyz="${x} ${y} ${z}" rpy="${R} ${P} ${Y}" />
+      <parent link="${namespace}/motion_sensor" />
+      <child link="${namespace}/${name}" />
+    </joint>
   </xacro:macro>
 </robot>

File: urdf/sensors/pano_array.xacro (robot description, xacro)
@@ -1,10 +1,10 @@
 <?xml version="1.0"?>
 <robot xmlns:xacro="http://ros.org/wiki/xacro">
-  <xacro:macro name="ben_pano_array" params="name x:=0.0 y:=0 z:=0.0 R:=0 P:=0 Y:=0 update_rate:=5">
+  <xacro:macro name="pano_array" params="name x:=0.0 y:=0 z:=0.0 R:=0 P:=0 Y:=0">
     <link name="${namespace}/${name}">
-      <visual name="${name}_visual">
+      <visual name="${name}_base_visual">
         <origin xyz="0 0 0" rpy="0 0 0"/>
         <geometry>
-          <mesh filename="package://ben_gazebo/models/meshes/panoramic_camera_housing.dae"/>
+          <mesh filename="package://ben_description/models/meshes/panoramic_camera_housing.dae"/>
         </geometry>
       </visual>
@@ -15,5 +15,4 @@
         </geometry>
       </collision>
-      <!-- Model inertia as box with <size>0.078 0.03 0.03</size> -->
       <inertial>
         <mass value="0.3"/>
@@ -27,12 +26,12 @@
       </inertial>
     </link>
-    <joint name="${namespace}/motion_sensor_to_${name}_joint" type="fixed">
+    <joint name="${namespace}/motion_sensor_to_${name}_base_joint" type="fixed">
       <origin xyz="${x} ${y} ${z}" rpy="${R} ${P} ${Y}" />
-      <parent link="${namespace}/motion_sensor_link" />
+      <parent link="${namespace}/motion_sensor" />
       <child link="${namespace}/${name}" />
     </joint>
-    <xacro:include filename="$(find ben_gazebo)/urdf/sensors/ben_pano_camera.xacro" />
+    <xacro:include filename="$(find ben_description)/urdf/sensors/pano_camera.xacro" />
     <xacro:macro name="loop" params="i">
-      <xacro:ben_pano_camera name="${name}" number="${i}" x="0.08" z="0.05" Y="${-radians(i*60)}" />
+      <xacro:pano_camera name="${name}" number="${i}" x="0.08" z="0.05" Y="${-radians(i*60)}" />
       <xacro:if value="${i}">
         <xacro:loop i="${i-1}" />

File: urdf/sensors/pano_camera.xacro (robot description, xacro)
@@ -1,11 +1,11 @@
 <?xml version="1.0"?>
 <robot xmlns:xacro="http://ros.org/wiki/xacro">
-  <xacro:macro name="ben_pano_camera" params="name number x:=0.1 y:=0 z:=0 R:=0 P:=0 Y:=0 update_rate:=5">
+  <xacro:macro name="pano_camera" params="name number x:=0.1 y:=0 z:=0 R:=0 P:=0 Y:=0">
     <!-- Monocular Camera -->
     <link name="${namespace}/${name}_${number}">
       <visual name="${name}_${number}_visual">
-        <origin xyz="-0.033 0 0" rpy="0 0 ${pi/2}"/>
+        <origin xyz="0.018 0 0" rpy="0 ${pi/2} 0"/>
         <geometry>
-          <mesh filename="package://vrx_gazebo/models/mono_camera/mesh/mono_camera.dae"/>
+          <cylinder radius="0.015" length="0.042"/>
         </geometry>
       </visual>
@@ -14,10 +14,4 @@
         <geometry>
           <cylinder radius="0.015" length="0.042"/>
-        </geometry>
-      </collision>
-      <collision name="${name}_box_collision">
-        <origin xyz="-0.0205 0 0" rpy="0 0 0"/>
-        <geometry>
-          <box size="0.036 0.03 0.03"/>
         </geometry>
       </collision>
@@ -67,44 +61,4 @@
       <child link="${namespace}/${name}_${number}_optical_rviz_mesh" />
     </joint>
-    <!-- Gazebo camera setup -->
-    <gazebo reference="${namespace}/${name}_${number}">
-      <sensor type="camera" name="${name}_${number}_sensor">
-        <update_rate>${update_rate}</update_rate>
-        <camera name="${name}_${number}_camera">
-          <horizontal_fov>1.26</horizontal_fov>
-          <image>
-            <width>2560</width>
-            <height>1440</height>
-            <format>R8G8B8</format>
-          </image>
-          <clip>
-            <near>0.05</near>
-            <far>5000</far>
-          </clip>
-          <noise>
-            <type>gaussian</type>
-            <!-- Noise is sampled independently per pixel on each frame.
-                 That pixel's noise value is added to each of its color
-                 channels, which at that point lie in the range [0,1]. -->
-            <mean>0.0</mean>
-            <stddev>0.007</stddev>
-          </noise>
-        </camera>
-        <plugin name="camera_plugin_${name}" filename="libgazebo_ros_camera.so">
-          <alwaysOn>true</alwaysOn>
-          <updateRate>0.0</updateRate>
-          <cameraName>${namespace}/${sensor_namespace}${camera_namespace}${name}_${number}</cameraName>
-          <imageTopicName>image_raw</imageTopicName>
-          <cameraInfoTopicName>camera_info</cameraInfoTopicName>
-          <frameName>${namespace}/${name}_${number}_optical</frameName>
-          <hackBaseline>0.07</hackBaseline>
-          <distortionK1>0.0</distortionK1>
-          <distortionK2>0.0</distortionK2>
-          <distortionK3>0.0</distortionK3>
-          <distortionT1>0.0</distortionT1>
-          <distortionT2>0.0</distortionT2>
-        </plugin>
-      </sensor>
-    </gazebo>
   </xacro:macro>
 </robot>

Commit message: Move pano and hide radar for simulation

File: urdf/ben_mesh.xacro (robot description, xacro)
@@ -58,5 +58,7 @@
   <xacro:ben_radar name="radar" x="-1.8" y="0.0" z="1.3"/>
   <xacro:include filename="$(find ben_description)/urdf/sensors/pano_array.xacro" />
-  <xacro:pano_array name="pano" x="-1.98" z="1.266"/>
+  <!-- <xacro:pano_array name="pano" x="-1.98" z="1.266"/> -->
+  <!-- HACK moved pano array up so light is not in field of view -->
+  <xacro:pano_array name="pano" x="-1.98" z="1.366"/>
   <xacro:include filename="$(find ben_description)/urdf/sensors/oem_gps.xacro" />
   <xacro:oem_gps name="gps" x="-0.953" y="0.103" z="0.628"/>

File: urdf/sensors/radar.xacro (robot description, xacro)
@@ -8,5 +8,5 @@
         <origin xyz="0 0 0" rpy="0 0 0"/>
         <geometry>
-          <cylinder radius="0.3" length="0.25"/>
+          <!-- <cylinder radius="0.3" length="0.25"/> -->
         </geometry>
       </visual>
